File: Arduino/hardware/RRAT-REV19/RRAT.sch (KiCad schematic (older format))
At the start: 39 parts, among them IC1 ATMEGA168-AU, J1 Conn_01x06, J2 Conn_02x03_Odd_Even, J3 Conn_02x20_Odd_Even, J4 Conn_01x12, Q1 32768Hz, U1 RFM26, U2 MIC94092

Commit message: Revert "rrat updates"
This reverts commit 8fcb23e6e4f1bd747ced1507a82f3c989f170f02.
Parts:
- removed C13: 100nF, RRAT Consolidated:C0603, symbol RRAT_consolidated:C
- removed D1: LED, symbol Device:LED
- removed R6: 470 (Provisional), symbol Device:R
- removed U2: MIC94092, symbol rrat:MIC94092
Connections:
- net labels added: IO_POWER_UP, LDR, RESET, SCL, SDA, VCC_0
- net labels removed: +3V3, ~RESET, ~SHUTDOWN
- wire segments 197 -> 177
- no-connect marks 27 -> 0
Other:
- note added: "Copyright: Bo Herrmannsen 2018"
- note removed: "As close to MIC94092\npin 4 as possible\n"
- note removed: "Copyright: Bo Herrmannsen 2018, Deniz Erbilgin 2019"
- note removed: "FTDI"
- note removed: "ICSP"
- note removed: "Pin Breakouts"
- moved on the sheet: C10

Commit message: rrat updates
Parts:
- added C13: 100nF, RRAT Consolidated:C0603, symbol RRAT_consolidated:C
- added D1: LED, symbol Device:LED
- added R6: 470 (Provisional), symbol Device:R
- added U2: MIC94092, symbol rrat:MIC94092
Connections:
- net labels added: +3V3, ~RESET, ~SHUTDOWN
- net labels removed: IO_POWER_UP, LDR, RESET, SCL, SDA, VCC_0
- wire segments 177 -> 197
- no-connect marks 0 -> 27
Other:
- note added: "As close to MIC94092\npin 4 as possible\n"
- note added: "Copyright: Bo Herrmannsen 2018, Deniz Erbilgin 2019"
- note added: "FTDI"
- note added: "ICSP"
- note added: "Pin Breakouts"
- note removed: "Copyright: Bo Herrmannsen 2018"
- moved on the sheet: C10
