File: Arduino/hardware/RRAT-REV19/RRAT.sch (KiCad schematic (older format))
At the start: 35 parts, among them IC1 ATMEGA168-AU, J1 Conn_01x06, J2 Conn_02x03_Odd_Even, J3 Conn_02x20_Odd_Even, J4 Conn_01x12, Q1 32768Hz, U1 RFM26

Commit message: RRAT update
Parts:
- R18: value 1K -> 1R
Connections:
- wire segments 177 -> 180
Other:
- moved on the sheet: C3, J3, R10, R12, R13, R14, R15, R16, R17, R18

Commit message: Fixed most DRC
Connections:
- net labels added: +3V3
- net labels removed: IO_POWER_UP, LDR, SCL, SDA, VCC_0
- wire segments 180 -> 189
- no-connect marks 0 -> 29
Other:
- note added: "Caps C2, C3 and C4 should be placed\nas close to the pins as possible and have\na via to ground as close as possible."
- note added: "Caps C5, C6, C7, C8, C9 and C10 should\nbe placed as close to the pins as possible\nand have a via to ground as close as possible."
- moved on the sheet: ANT1, C1, C10, C11, C12, C4, C5, C6, C7, C8, C9, IC1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

Commit message: Added switch
Parts:
- added C13: 0nF, RRAT Consolidated:C0603, symbol RRAT_consolidated:C
- added C14: 100nF, RRAT Consolidated:C0603, symbol RRAT_consolidated:C
- added U2: MIC94092, symbol RRAT_consolidated:MIC9409x
- C10, C7, C8, C9: value 47 pF -> 47pF
Connections:
- net labels added: ~SHUTDOWN
- wire segments 189 -> 205
- no-connect marks 29 -> 27
Other:
- note added: "Caps C13* and C14 should be placed\nas close to the pins as possible and have\na via to ground as close as possible.\n\n*C13 should not be fitted."
- note added: "NOTE:\nSpecial considerations on placement\nand keepouts.\n\nSee existing designs."
- moved on the sheet: C1, C11, C12, C2, C3, C4, IC1, J1, J4, JP1, Q1, R1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
